File: CC45.kicad_pcb (KiCad board)
At the start: 2 copper layers, 247 x 80.8 mm, 122 parts, among them J1 AVR-ISP-6, SW1 SW_Push_Dual, SW10 K08, SW11 K09, SW12 K0A, SW13 K0B, SW14 K0C, SW15 K10, SW16 K11, SW17 K12, SW18 K13, SW19 K14, SW2 K00, SW20 K15, SW21 K16, SW22 K17, SW23 K18, SW24 K19, SW25 K1A, SW26 K1B, SW27 K20, SW28 K21, SW29 K22, SW3 K01, SW30 K23, SW31 K24, SW32 K25, SW33 K26, SW34 K27, SW35 K28, SW36 K29, SW37 K2A, SW38 K2B, SW39 K30, SW4 K02, SW40 K31, SW41 K32, SW42 K33, SW43 K34, SW44 K36, SW45 K38, SW46 K39, SW47 K3A, SW48 K3B, SW5 K03, SW6 K04, SW7 K05, SW8 K06, SW9 K07, U1 ATmega32U4-AU, U2 PRTR5V0U2X, X1 XTAL

Commit message: moved values on silkscreen to make them more visible
Parts:
- SW1: value SW_Push_Dual -> RESET
Changed lines of the file:
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@@
       (effects (font (size 1 1) (thickness 0.15)) (justify mirror))
     )
-    (fp_text user "MOSI" (at 4.45 -1 -90) (layer "B.SilkS")
+    (fp_text user "MOSI" (at 4.45 -0.75 -90) (layer "B.SilkS")
       (effects (font (size 1 1) (thickness 0.15)) (justify mirror))
     )
@@
       (effects (font (size 1 1) (thickness 0.15)))
     )
-    (fp_text value "SW_Push_Dual" (at 0 -3.5625) (layer "B.SilkS")
+    (fp_text value "RESET" (at 0.75 -3.4) (layer "B.SilkS")
       (effects (font (size 1 1) (thickness 0.15)) (justify mirror))
     )
@@
     (tags "resistor handsolder")
     (attr smd)
-    (fp_text reference "R6" (at 0 1.82 90) (layer "B.SilkS")
+    (fp_text reference "R6" (at 3.3 -0.05 180) (layer "B.SilkS")
       (effects (font (size 1 1) (thickness 0.15)) (justify mirror))
     )
@@
     (tags "SOD-323")
     (attr smd)
-    (fp_text reference "D41" (at 0 1.85 90) (layer "B.SilkS")
+    (fp_text reference "D41" (at 0 -1.5375 90) (layer "B.SilkS")
       (effects (font (size 1 1) (thickness 0.15)) (justify mirror))
     )
@@
     (tags "SOD-323")
     (attr smd)
-    (fp_text reference "D6" (at 0 1.7285 270) (layer "B.SilkS")
+    (fp_text reference "D6" (at 0.05 -1.5625 270) (layer "B.SilkS")
       (effects (font (size 1 1) (thickness 0.15)) (justify mirror))
     )
@@
     (tags "capacitor handsolder")
     (attr smd)
-    (fp_text reference "C3" (at 0 1.82 90) (layer "B.SilkS")
+    (fp_text reference "C3" (at -0.65 -1.85 90) (layer "B.SilkS")
       (effects (font (size 1 1) (thickness 0.15)) (justify mirror))
     )
@@
   (gr_arc (start 24.9375 98.5625) (end 23.75 98.5625) (angle -90) (layer "Edge.Cuts") (width 0.15))
   (gr_arc (start 24.9375 24.9375) (end 24.9375 23.75) (angle -90) (layer "Edge.Cuts") (width 0.15))
+  (segment (start 48.6875 73.25) (end 48.6875 72.5) (width 0.25) (layer "B.Cu") (net 34))
+  (segment (start 137.7 81.9) (end 137 81.2) (width 0.25) (layer "B.Cu") (net 34))
+  (segment (start 137 81.2) (end 137 80.65) (width 0.25) (layer "B.Cu") (net 34))
+  (segment (start 138.8 81.9) (end 137.7 81.9) (width 0.25) (layer "B.Cu") (net 34))
+  (segment (start 137 80.65) (end 133.05 76.7) (width 0.25) (layer "B.Cu") (net 34))
+  (segment (start 133.05 76.7) (end 52.1375 76.7) (width 0.25) (layer "B.Cu") (net 34))
+  (segment (start 52.1375 76.7) (end 48.6875 73.25) (width 0.25) (layer "B.Cu") (net 34))
+  (segment (start 137.85 82.7) (end 136.55 81.4) (width 0.25) (layer "B.Cu") (net 67))
+  (segment (start 138.8 82.7) (end 137.85 82.7) (width 0.25) (layer "B.Cu") (net 67))
+  (segment (start 37.130685 76.885) (end 36.565 76.885) (width 0.25) (layer "B.Cu") (net 67))
+  (segment (start 136.55 81.4) (end 136.55 80.85) (width 0.25) (layer "B.Cu") (net 67))
+  (segment (start 136.55 80.85) (end 132.85 77.15) (width 0.25) (layer "B.Cu") (net 67))
+  (segment (start 132.85 77.15) (end 37.395685 77.15) (width 0.25) (layer "B.Cu") (net 67))
+  (segment (start 37.395685 77.15) (end 37.130685 76.885) (width 0.25) (layer "B.Cu") (net 67))
+  (segment (start 43.65 54.55) (end 43.9375 54.2625) (width 0.25) (layer "B.Cu") (net 21))
+  (segment (start 39.15 54.55) (end 43.65 54.55) (width 0.25) (layer "B.Cu") (net 21))
+  (segment (start 33.5 75.3) (end 33.5 60.2) (width 0.25) (layer "B.Cu") (net 21))
+  (segment (start 33.5 60.2) (end 39.15 54.55) (width 0.25) (layer "B.Cu") (net 21))
+  (segment (start 138.8 83.5) (end 137.968224 83.5) (width 0.25) (layer "B.Cu") (net 21))
+  (segment (start 136.05 81.581776) (end 136.05 81) (width 0.25) (layer "B.Cu") (net 21))
+  (segment (start 136.05 81) (end 132.660001 77.610001) (width 0.25) (layer "B.Cu") (net 21))
+  (segment (start 132.660001 77.610001) (end 35.810001 77.610001) (width 0.25) (layer "B.Cu") (net 21))
+  (segment (start 43.9375 54.2625) (end 43.9375 53.5) (width 0.25) (layer "B.Cu") (net 21))
+  (segment (start 137.968224 83.5) (end 136.05 81.581776) (width 0.25) (layer "B.Cu") (net 21))
+  (segment (start 35.810001 77.610001) (end 33.5 75.3) (width 0.25) (layer "B.Cu") (net 21))
   (segment (start 137.55 77.9) (end 135.075 75.425) (width 0.25) (layer "B.Cu") (net 62))
   (segment (start 138.8 77.9) (end 137.55 77.9) (width 0.25) (layer "B.Cu") (net 62))
@@
   (segment (start 64.3 76.25) (end 63.099999 75.049999) (width 0.25) (layer "B.Cu") (net 68))
   (segment (start 63.099999 75.049999) (end 62.7 74.65) (width 0.25) (layer "B.Cu") (net 68))
-  (segment (start 52.1375 76.7) (end 48.6875 73.25) (width 0.25) (layer "B.Cu") (net 34))
-  (segment (start 133.05 76.7) (end 52.1375 76.7) (width 0.25) (layer "B.Cu") (net 34))
-  (segment (start 137 80.65) (end 133.05 76.7) (width 0.25) (layer "B.Cu") (net 34))
-  (segment (start 137 81.2) (end 137 80.65) (width 0.25) (layer "B.Cu") (net 34))
-  (segment (start 138.8 81.9) (end 137.7 81.9) (width 0.25) (layer "B.Cu") (net 34))
-  (segment (start 137.7 81.9) (end 137 81.2) (width 0.25) (layer "B.Cu") (net 34))
-  (segment (start 48.6875 73.25) (end 48.6875 72.5) (width 0.25) (layer "B.Cu") (net 34))
-  (segment (start 37.395685 77.15) (end 37.130685 76.885) (width 0.25) (layer "B.Cu") (net 67))
-  (segment (start 132.85 77.15) (end 37.395685 77.15) (width 0.25) (layer "B.Cu") (net 67))
-  (segment (start 136.55 80.85) (end 132.85 77.15) (width 0.25) (layer "B.Cu") (net 67))
-  (segment (start 136.55 81.4) (end 136.55 80.85) (width 0.25) (layer "B.Cu") (net 67))
-  (segment (start 138.8 82.7) (end 137.85 82.7) (width 0.25) (layer "B.Cu") (net 67))
-  (segment (start 137.85 82.7) (end 136.55 81.4) (width 0.25) (layer "B.Cu") (net 67))
-  (segment (start 37.130685 76.885) (end 36.565 76.885) (width 0.25) (layer "B.Cu") (net 67))
-  (segment (start 35.810001 77.610001) (end 33.5 75.3) (width 0.25) (layer "B.Cu") (net 21))
-  (segment (start 132.660001 77.610001) (end 35.810001 77.610001) (width 0.25) (layer "B.Cu") (net 21))
-  (segment (start 136.05 81) (end 132.660001 77.610001) (width 0.25) (layer "B.Cu") (net 21))
-  (segment (start 136.05 81.581776) (end 136.05 81) (width 0.25) (layer "B.Cu") (net 21))
-  (segment (start 138.8 83.5) (end 137.968224 83.5) (width 0.25) (layer "B.Cu") (net 21))
-  (segment (start 39.15 54.55) (end 43.65 54.55) (width 0.25) (layer "B.Cu") (net 21))
-  (segment (start 137.968224 83.5) (end 136.05 81.581776) (width 0.25) (layer "B.Cu") (net 21))
-  (segment (start 33.5 75.3) (end 33.5 60.2) (width 0.25) (layer "B.Cu") (net 21))
-  (segment (start 33.5 60.2) (end 39.15 54.55) (width 0.25) (layer "B.Cu") (net 21))
-  (segment (start 43.9375 54.2625) (end 43.9375 53.5) (width 0.25) (layer "B.Cu") (net 21))
-  (segment (start 43.65 54.55) (end 43.9375 54.2625) (width 0.25) (layer "B.Cu") (net 21))
   (segment (start 35.6236 78.06001) (end 29.344999 71.781409) (width 0.25) (layer "B.Cu") (net 7))
   (segment (start 132.46001 78.06001) (end 35.6236 78.06001) (width 0.25) (layer "B.Cu") (net 7))
