File: CC45.kicad_pcb (KiCad board)
At the start: 2 copper layers, 247 x 80.8 mm, 130 parts, among them J1 AVR-ISP-6, SW1 RESET, SW10 K08, SW11 K09, SW12 K0A, SW13 K0B, SW14 K0C, SW15 K10, SW16 K11, SW17 K12, SW18 K13, SW19 K14, SW2 K00, SW20 K15, SW21 K16, SW22 K17, SW23 K18, SW24 K19, SW25 K1A, SW26 K1B, SW27 K20, SW28 K21, SW29 K22, SW3 K01, SW30 K23, SW31 K24, SW32 K25, SW33 K26, SW34 K27, SW35 K28, SW36 K29, SW37 K2A, SW38 K2B, SW39 K30, SW4 K02, SW40 K31, SW41 K32, SW42 K33, SW43 K34, SW44 K36, SW45 K38, SW46 K39, SW47 K3A, SW48 K3B, SW5 K03, SW6 K04, SW7 K05, SW8 K06, SW9 K07, U1 ATmega32U4-AU, U2 PRTR5V0U2X, X1 XTAL

Commit message: Updated version written on pcb
Other:
- board text added: "CC45 v2.1 by Druz github.com/aaarsene/CC45"
- board text removed: "CC45 v2 by Druz github.com/aaarsene/CC45"

Commit message: Remove usb port and safeties, add jst connector
Parts:
- removed F1: 500m, Fuse:Fuse_1206_3216Metric_Pad1.42x1.75mm_HandSolder
- removed G***: LOGO, cc:cc
- removed R5, R6: 5.1k, Resistor_SMD:R_1206_3216Metric_Pad1.42x1.75mm_HandSolder
- removed REF** (x5): MountingHole_2.2mm_M2_Pad, MountingHole:MountingHole_2.2mm_M2_Pad
- removed U2: PRTR5V0U2X, random-keyboard-parts:SOT143B
- removed USB1: HRO-TYPE-C-31-M-12, Type-C:HRO-TYPE-C-31-M-12-HandSoldering
- added J2: Conn_01x04, random-keyboard-parts:JST-SR-4, B.Cu at (87.2, 42.8)
- moved D7 10.9 mm to (149.6, 36.8)
- moved D4 6.39 mm to (92.6, 36.8)
- moved D5 6.39 mm to (111.6, 36.8)
- moved D6 6.39 mm to (130.6, 36.8)
Connections:
- R2 pad 2: /USB_N -> /D_N
- R3 pad 2: /USB_P -> /D_P
Routing:
- net /USB_N: track 130.2 -> 0.00 mm
- net /USB_P: track 128.4 -> 0.00 mm
- net GND: track 308.7 -> 188.0 mm, vias 2 -> 0
- net +5V: track 222.4 -> 150.9 mm, vias 8 -> 7
- net /D_N: track 0.00 -> 42.0 mm
- net /D_P: track 0.00 -> 41.3 mm
- net VCC: track 17.8 -> 0.00 mm
- net Net-(R6-Pad2): track 12.2 -> 0.00 mm
- net Net-(R5-Pad2): track 6.96 -> 0.00 mm, vias 2 -> 0
- net Net-(D7-Pad2): track 14.3 -> 7.46 mm
- net row0: track 283.5 -> 278.3 mm, vias 2 -> 0
- net Net-(D6-Pad2): track 9.21 -> 7.46 mm
- net Net-(D5-Pad2): track 9.21 -> 7.46 mm
- net Net-(D4-Pad2): track 9.21 -> 7.46 mm
Other:
- board size 247 x 80.8 mm -> 247 x 76 mm

Commit message: Update step
Other:
- rule pad_to_mask_clearance: 0.051 -> 0
- board text added: "CC45 v2.1-jst by Druz github.com/aaarsene/CC45"
- board text removed: "CC45 v2.1 by Druz github.com/aaarsene/CC45"
