File: matrix.sch (KiCad schematic (older format))
At the start: 94 parts, among them SW10 K08, SW11 K09, SW12 K0A, SW13 K0B, SW14 K0C, SW15 K10, SW16 K11, SW17 K12, SW18 K13, SW19 K14, SW2 K00, SW20 K15, SW21 K16, SW22 K17, SW23 K18, SW24 K19, SW25 K1A, SW26 K1B, SW27 K20, SW28 K21, SW29 K22, SW3 K01, SW30 K23, SW31 K24, SW32 K25, SW33 K26, SW34 K27, SW35 K28, SW36 K29, SW37 K2A, SW38 K2B, SW39 K30, SW4 K02, SW40 K31, SW41 K32, SW42 K33, SW43 K34, SW44 K36, SW45 K38, SW46 K39, SW47 K3A, SW48 K3B, SW5 K03, SW6 K04, SW7 K05, SW8 K06, SW9 K07

Commit message: Placed footprints on pcb and routed everything except the matrix
Parts:
- SW10, SW11, SW12, SW13, SW14, SW16, SW17, SW18, SW19, SW2, SW20, SW21, SW22, SW23, SW24, SW25, SW28, SW29, SW3, SW30, SW31, SW32, SW33, SW34, SW35, SW36, SW37, SW4, SW40, SW47, SW5, SW6, SW7, SW8, SW9: footprint MX_19mm:MX_19mm-1U -> MX_19mm:MX_19mm-1U-NoLED
- SW15, SW38, SW39, SW41, SW42, SW45, SW46, SW48: footprint MX_19mm:MX_19mm-1.25U -> MX_19mm:MX_19mm-1.25U-NoLED
- SW26, SW27, SW43, SW44: footprint MX_19mm:MX_19mm-1.75U -> MX_19mm:MX_19mm-1.75U-NoLED

Commit message: moving C4 closer to the mcu and adding JLC parts numbers
Parts:
- D1, D10, D11, D12, D13, D14, D15, D16, D17, D18, D19, D2, D20, D21, D22, D23, D24, D25, D26, D27, D28, D29, D3, D30, D31, D32, D33, D34, D35, D36, D37, D38, D39, D4, D40, D41, D42, D43, D44, D45, D46, D47, D5, D6, D7, D8, D9: LCSC (none) -> C84063
Changed lines of the file:
@@
 F 2 "Diode_SMD:D_SOD-323_HandSoldering" H 1975 1600 50  0001 C CNN
 F 3 "~" H 1975 1600 50  0001 C CNN
+F 4 "C84063" H 1975 1600 50  0001 C CNN "LCSC"
 	1    1975 1600
 	0    -1   -1   0
@@
 F 2 "Diode_SMD:D_SOD-323_HandSoldering" H 3025 1600 50  0001 C CNN
 F 3 "~" H 3025 1600 50  0001 C CNN
+F 4 "C84063" H 3025 1600 50  0001 C CNN "LCSC"
 	1    3025 1600
 	0    -1   -1   0
@@
 F 2 "Diode_SMD:D_SOD-323_HandSoldering" H 2500 1600 50  0001 C CNN
 F 3 "~" H 2500 1600 50  0001 C CNN
+F 4 "C84063" H 2500 1600 50  0001 C CNN "LCSC"
 	1    2500 1600
 	0    -1   -1   0
@@
 F 2 "Diode_SMD:D_SOD-323_HandSoldering" H 5125 1600 50  0001 C CNN
 F 3 "~" H 5125 1600 50  0001 C CNN
+F 4 "C84063" H 5125 1600 50  0001 C CNN "LCSC"
 	1    5125 1600
 	0    -1   -1   0
@@
 F 2 "Diode_SMD:D_SOD-323_HandSoldering" H 4600 1600 50  0001 C CNN
 F 3 "~" H 4600 1600 50  0001 C CNN
+F 4 "C84063" H 4600 1600 50  0001 C CNN "LCSC"
 	1    4600 1600
 	0    -1   -1   0
@@
 F 2 "Diode_SMD:D_SOD-323_HandSoldering" H 4075 1600 50  0001 C CNN
 F 3 "~" H 4075 1600 50  0001 C CNN
+F 4 "C84063" H 4075 1600 50  0001 C CNN "LCSC"
 	1    4075 1600
 	0    -1   -1   0
@@
 F 2 "Diode_SMD:D_SOD-323_HandSoldering" H 3550 1600 50  0001 C CNN
 F 3 "~" H 3550 1600 50  0001 C CNN
+F 4 "C84063" H 3550 1600 50  0001 C CNN "LCSC"
 	1    3550 1600
 	0    -1   -1   0
@@
 F 2 "Diode_SMD:D_SOD-323_HandSoldering" H 7225 1600 50  0001 C CNN
 F 3 "~" H 7225 1600 50  0001 C CNN
+F 4 "C84063" H 7225 1600 50  0001 C CNN "LCSC"
 	1    7225 1600
 	0    -1   -1   0
@@
 F 2 "Diode_SMD:D_SOD-323_HandSoldering" H 6700 1600 50  0001 C CNN
 F 3 "~" H 6700 1600 50  0001 C CNN
+F 4 "C84063" H 6700 1600 50  0001 C CNN "LCSC"
 	1    6700 1600
 	0    -1   -1   0
@@
 F 2 "Diode_SMD:D_SOD-323_HandSoldering" H 5650 1600 50  0001 C CNN
 F 3 "~" H 5650 1600 50  0001 C CNN
+F 4 "C84063" H 5650 1600 50  0001 C CNN "LCSC"
 	1    5650 1600
 	0    -1   -1   0
@@
 F 2 "Diode_SMD:D_SOD-323_HandSoldering" H 7750 1600 50  0001 C CNN
 F 3 "~" H 7750 1600 50  0001 C CNN
+F 4 "C84063" H 7750 1600 50  0001 C CNN "LCSC"
 	1    7750 1600
 	0    -1   -1   0
@@
 F 2 "Diode_SMD:D_SOD-323_HandSoldering" H 3025 2400 50  0001 C CNN
 F 3 "~" H 3025 2400 50  0001 C CNN
+F 4 "C84063" H 3025 2400 50  0001 C CNN "LCSC"
 	1    3025 2400
 	0    -1   -1   0
@@
 F 2 "Diode_SMD:D_SOD-323_HandSoldering" H 2500 2400 50  0001 C CNN
 F 3 "~" H 2500 2400 50  0001 C CNN
+F 4 "C84063" H 2500 2400 50  0001 C CNN "LCSC"
 	1    2500 2400
 	0    -1   -1   0
@@
 F 2 "Diode_SMD:D_SOD-323_HandSoldering" H 1975 2400 50  0001 C CNN
 F 3 "~" H 1975 2400 50  0001 C CNN
+F 4 "C84063" H 1975 2400 50  0001 C CNN "LCSC"
 	1    1975 2400
 	0    -1   -1   0
@@
 F 2 "Diode_SMD:D_SOD-323_HandSoldering" H 5125 2400 50  0001 C CNN
 F 3 "~" H 5125 2400 50  0001 C CNN
+F 4 "C84063" H 5125 2400 50  0001 C CNN "LCSC"
 	1    5125 2400
 	0    -1   -1   0
@@
 F 2 "Diode_SMD:D_SOD-323_HandSoldering" H 1450 2400 50  0001 C CNN
 F 3 "~" H 1450 2400 50  0001 C CNN
+F 4 "C84063" H 1450 2400 50  0001 C CNN "LCSC"
 	1    1450 2400
 	0    -1   -1   0
@@
 F 2 "Diode_SMD:D_SOD-323_HandSoldering" H 4600 2400 50  0001 C CNN
 F 3 "~" H 4600 2400 50  0001 C CNN
+F 4 "C84063" H 4600 2400 50  0001 C CNN "LCSC"
 	1    4600 2400
 	0    -1   -1   0
@@
 F 2 "Diode_SMD:D_SOD-323_HandSoldering" H 7225 2400 50  0001 C CNN
 F 3 "~" H 7225 2400 50  0001 C CNN
+F 4 "C84063" H 7225 2400 50  0001 C CNN "LCSC"
 	1    7225 2400
 	0    -1   -1   0
@@
 F 2 "Diode_SMD:D_SOD-323_HandSoldering" H 6175 2400 50  0001 C CNN
 F 3 "~" H 6175 2400 50  0001 C CNN
+F 4 "C84063" H 6175 2400 50  0001 C CNN "LCSC"
 	1    6175 2400
 	0    -1   -1   0
@@
 F 2 "Diode_SMD:D_SOD-323_HandSoldering" H 5650 2400 50  0001 C CNN
 F 3 "~" H 5650 2400 50  0001 C CNN
+F 4 "C84063" H 5650 2400 50  0001 C CNN "LCSC"
 	1    5650 2400
 	0    -1   -1   0
@@
 F 2 "Diode_SMD:D_SOD-323_HandSoldering" H 4075 2400 50  0001 C CNN
 F 3 "~" H 4075 2400 50  0001 C CNN
+F 4 "C84063" H 4075 2400 50  0001 C CNN "LCSC"
 	1    4075 2400
 	0    -1   -1   0
@@
 F 2 "Diode_SMD:D_SOD-323_HandSoldering" H 3550 2400 50  0001 C CNN
 F 3 "~" H 3550 2400 50  0001 C CNN
+F 4 "C84063" H 3550 2400 50  0001 C CNN "LCSC"
 	1    3550 2400
 	0    -1   -1   0
@@
 F 2 "Diode_SMD:D_SOD-323_HandSoldering" H 6700 2400 50  0001 C CNN
 F 3 "~" H 6700 2400 50  0001 C CNN
+F 4 "C84063" H 6700 2400 50  0001 C CNN "LCSC"
 	1    6700 2400
 	0    -1   -1   0
@@
 F 2 "Diode_SMD:D_SOD-323_HandSoldering" H 3025 3200 50  0001 C CNN
 F 3 "~" H 3025 3200 50  0001 C CNN
+F 4 "C84063" H 3025 3200 50  0001 C CNN "LCSC"
 	1    3025 3200
 	0    -1   -1   0
@@
 F 2 "Diode_SMD:D_SOD-323_HandSoldering" H 2500 3200 50  0001 C CNN
 F 3 "~" H 2500 3200 50  0001 C CNN
+F 4 "C84063" H 2500 3200 50  0001 C CNN "LCSC"
 	1    2500 3200
 	0    -1   -1   0
@@
 F 2 "Diode_SMD:D_SOD-323_HandSoldering" H 1975 3200 50  0001 C CNN
 F 3 "~" H 1975 3200 50  0001 C CNN
+F 4 "C84063" H 1975 3200 50  0001 C CNN "LCSC"
 	1    1975 3200
 	0    -1   -1   0
@@
 F 2 "Diode_SMD:D_SOD-323_HandSoldering" H 5125 3200 50  0001 C CNN
 F 3 "~" H 5125 3200 50  0001 C CNN
+F 4 "C84063" H 5125 3200 50  0001 C CNN "LCSC"
 	1    5125 3200
 	0    -1   -1   0
@@
 F 2 "Diode_SMD:D_SOD-323_HandSoldering" H 1450 3200 50  0001 C CNN
 F 3 "~" H 1450 3200 50  0001 C CNN
+F 4 "C84063" H 1450 3200 50  0001 C CNN "LCSC"
 	1    1450 3200
 	0    -1   -1   0
@@
 F 2 "Diode_SMD:D_SOD-323_HandSoldering" H 4600 3200 50  0001 C CNN
 F 3 "~" H 4600 3200 50  0001 C CNN
+F 4 "C84063" H 4600 3200 50  0001 C CNN "LCSC"
 	1    4600 3200
 	0    -1   -1   0
@@
 F 2 "Diode_SMD:D_SOD-323_HandSoldering" H 7225 3200 50  0001 C CNN
 F 3 "~" H 7225 3200 50  0001 C CNN
+F 4 "C84063" H 7225 3200 50  0001 C CNN "LCSC"
 	1    7225 3200
 	0    -1   -1   0
@@
 F 2 "Diode_SMD:D_SOD-323_HandSoldering" H 6175 3200 50  0001 C CNN
 F 3 "~" H 6175 3200 50  0001 C CNN
+F 4 "C84063" H 6175 3200 50  0001 C CNN "LCSC"
 	1    6175 3200
 	0    -1   -1   0
@@
 F 2 "Diode_SMD:D_SOD-323_HandSoldering" H 5650 3200 50  0001 C CNN
 F 3 "~" H 5650 3200 50  0001 C CNN
+F 4 "C84063" H 5650 3200 50  0001 C CNN "LCSC"
 	1    5650 3200
 	0    -1   -1   0
@@
 F 2 "Diode_SMD:D_SOD-323_HandSoldering" H 4075 3200 50  0001 C CNN
 F 3 "~" H 4075 3200 50  0001 C CNN
+F 4 "C84063" H 4075 3200 50  0001 C CNN "LCSC"
 	1    4075 3200
 	0    -1   -1   0
@@
 F 2 "Diode_SMD:D_SOD-323_HandSoldering" H 3550 3200 50  0001 C CNN
 F 3 "~" H 3550 3200 50  0001 C CNN
+F 4 "C84063" H 3550 3200 50  0001 C CNN "LCSC"
 	1    3550 3200
 	0    -1   -1   0
@@
 F 2 "Diode_SMD:D_SOD-323_HandSoldering" H 6700 3200 50  0001 C CNN
 F 3 "~" H 6700 3200 50  0001 C CNN
+F 4 "C84063" H 6700 3200 50  0001 C CNN "LCSC"
 	1    6700 3200
 	0    -1   -1   0
@@
 F 2 "Diode_SMD:D_SOD-323_HandSoldering" H 3025 4000 50  0001 C CNN
 F 3 "~" H 3025 4000 50  0001 C CNN
+F 4 "C84063" H 3025 4000 50  0001 C CNN "LCSC"
 	1    3025 4000
 	0    -1   -1   0
@@
 F 2 "Diode_SMD:D_SOD-323_HandSoldering" H 2500 4000 50  0001 C CNN
 F 3 "~" H 2500 4000 50  0001 C CNN
+F 4 "C84063" H 2500 4000 50  0001 C CNN "LCSC"
 	1    2500 4000
 	0    -1   -1   0
@@
 F 2 "Diode_SMD:D_SOD-323_HandSoldering" H 1975 4000 50  0001 C CNN
 F 3 "~" H 1975 4000 50  0001 C CNN
+F 4 "C84063" H 1975 4000 50  0001 C CNN "LCSC"
 	1    1975 4000
 	0    -1   -1   0
@@
 F 2 "Diode_SMD:D_SOD-323_HandSoldering" H 1450 4000 50  0001 C CNN
 F 3 "~" H 1450 4000 50  0001 C CNN
+F 4 "C84063" H 1450 4000 50  0001 C CNN "LCSC"
 	1    1450 4000
 	0    -1   -1   0
@@
 F 2 "Diode_SMD:D_SOD-323_HandSoldering" H 4600 4000 50  0001 C CNN
 F 3 "~" H 4600 4000 50  0001 C CNN
+F 4 "C84063" H 4600 4000 50  0001 C CNN "LCSC"
 	1    4600 4000
 	0    -1   -1   0
@@
 F 2 "Diode_SMD:D_SOD-323_HandSoldering" H 7225 4000 50  0001 C CNN
 F 3 "~" H 7225 4000 50  0001 C CNN
+F 4 "C84063" H 7225 4000 50  0001 C CNN "LCSC"
 	1    7225 4000
 	0    -1   -1   0
@@
 F 2 "Diode_SMD:D_SOD-323_HandSoldering" H 6175 4000 50  0001 C CNN
 F 3 "~" H 6175 4000 50  0001 C CNN
+F 4 "C84063" H 6175 4000 50  0001 C CNN "LCSC"
 	1    6175 4000
 	0    -1   -1   0
@@
 F 2 "Diode_SMD:D_SOD-323_HandSoldering" H 5650 4000 50  0001 C CNN
 F 3 "~" H 5650 4000 50  0001 C CNN
+F 4 "C84063" H 5650 4000 50  0001 C CNN "LCSC"
 	1    5650 4000
 	0    -1   -1   0
@@
 F 2 "Diode_SMD:D_SOD-323_HandSoldering" H 3550 4000 50  0001 C CNN
 F 3 "~" H 3550 4000 50  0001 C CNN
+F 4 "C84063" H 3550 4000 50  0001 C CNN "LCSC"
 	1    3550 4000
 	0    -1   -1   0
@@
 F 2 "Diode_SMD:D_SOD-323_HandSoldering" H 6700 4000 50  0001 C CNN
 F 3 "~" H 6700 4000 50  0001 C CNN
+F 4 "C84063" H 6700 4000 50  0001 C CNN "LCSC"
 	1    6700 4000
 	0    -1   -1   0
@@
 F 2 "Diode_SMD:D_SOD-323_HandSoldering" H 1450 1600 50  0001 C CNN
 F 3 "~" H 1450 1600 50  0001 C CNN
+F 4 "C84063" H 1450 1600 50  0001 C CNN "LCSC"
 	1    1450 1600
 	0    -1   -1   0
@@
 F 2 "Diode_SMD:D_SOD-323_HandSoldering" H 6175 1600 50  0001 C CNN
 F 3 "~" H 6175 1600 50  0001 C CNN
+F 4 "C84063" H 6175 1600 50  0001 C CNN "LCSC"
 	1    6175 1600
 	0    -1   -1   0
